File: MCU logger - Huskies lab.kicad_sch (KiCad schematic)
At the start: 0 parts

Commit message: added the components required for the schematic
Parts:
- added BT?: Battery_Cell, symbol Device:Battery_Cell
- added C? (x4): C, symbol Device:C
- added C?: C_Polarized, symbol Device:C_Polarized
- added D? (x2): LED, symbol Device:LED
- added H? (x4): MountingHole, symbol Mechanical:MountingHole
- added R? (x7): R, symbol Device:R
- added U? (x2): 24LC1025, symbol Memory_EEPROM:24LC1025
- added U?: ATMEGA328P-AU, QFP80P900X900X120-32N, symbol ATMEGA328P-AU:ATMEGA328P-AU
- added U?: DS1337S+, SOIC127P600X175-8N, symbol DS1337S_:DS1337S+
- added Y? (x2): Crystal, symbol Device:Crystal
Connections:
- new net: U?.21 (GND), U?.3 (GND), U?.5 (GND)
- new net: U?.4 (VCC), U?.6 (VCC)
Other:
- added sheet connectors (connectors.kicad_sch)
